File: KiCAD/RGBLLSC.kicad_pcb (KiCad board)
At the start: 2 copper layers, 69.9 x 36.8 mm, 20 parts, among them P2 PWR IN, P3 MAIN OUT, Q1 FQP30N06L, Q2 FQP30N06L, Q3 FQP30N06L, SW1 SW_PUSH, U1 PIC12F1840

Commit message: Cleaned Project
Connections:
- SW1 pad 1: GND -> Net-(P1-Pad1)
- SW1 pad 4: (no net) -> GND
Routing:
- net GND: track 72.0 -> 67.2 mm
Changed lines of the file:
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@@
 (kicad_pcb (version 4) (host pcbnew 4.0.1-3.201512221402+6198~38~ubuntu14.04.1-stable)
   (general
-    (links 37)
-    (no_connects 5)
+    (links 38)
+    (no_connects 6)
     (area 99.975 67 210.997714 121.995001)
     (thickness 1.6)
     (drawings 12)
-    (tracks 108)
+    (tracks 106)
     (zones 0)
     (modules 20)
@@
   )
   (setup
-    (last_trace_width 0.25)
+    (last_trace_width 0.508)
     (user_trace_width 0.508)
     (user_trace_width 1.27)
@@
     (fp_line (start 6 2) (end 6 2) (layer F.SilkS) (width 0))
     (fp_circle (center 3 2) (end 4 3) (layer F.SilkS) (width 0))
-    (pad 4 thru_hole circle (at 6 4 90) (size 1.7 1.7) (drill 1) (layers *.Cu *.Mask))
+    (pad 4 thru_hole circle (at 6 4 90) (size 1.7 1.7) (drill 1) (layers *.Cu *.Mask)
+      (net 1 GND))
     (pad 3 thru_hole circle (at 0 4 90) (size 1.7 1.7) (drill 1) (layers *.Cu *.Mask)
       (net 1 GND))
@@
       (net 4 "Net-(P1-Pad1)"))
     (pad 1 thru_hole circle (at 0 0 90) (size 1.7 1.7) (drill 1) (layers *.Cu *.Mask)
-      (net 1 GND))
+      (net 4 "Net-(P1-Pad1)"))
   )
   (module Housings_DIP:DIP-8_W7.62mm_LongPads (layer F.Cu)
@@
   (gr_line (start 173.99 116.84) (end 173.99 85.09) (angle 90) (layer Edge.Cuts) (width 0.15))
   (gr_line (start 173.99 85.09) (end 113.03 85.09) (angle 90) (layer Edge.Cuts) (width 0.15))
+  (segment (start 166.636 86.868) (end 166.636 87.642) (width 0.508) (layer F.Cu) (net 1) (status 400000))
+  (segment (start 169.639 88.265) (end 171.386 90.012) (width 0.508) (layer F.Cu) (net 1) (status 800000))
+  (segment (start 167.259 88.265) (end 169.639 88.265) (width 0.508) (layer F.Cu) (net 1))
+  (segment (start 166.636 87.642) (end 167.259 88.265) (width 0.508) (layer F.Cu) (net 1))
   (segment (start 149.225 96.901) (end 147.574 95.25) (width 0.508) (layer F.Cu) (net 1))
   (segment (start 147.574 95.25) (end 146.292 95.25) (width 0.508) (layer F.Cu) (net 1))
@@
   (segment (start 172.466 99.06) (end 172.466 107.696) (width 0.508) (layer F.Cu) (net 1))
   (segment (start 171.386 97.98) (end 172.466 99.06) (width 0.508) (layer F.Cu) (net 1))
-  (segment (start 166.636 86.868) (end 166.636 87.642) (width 0.508) (layer F.Cu) (net 1))
-  (segment (start 169.037 94.361) (end 167.386 96.012) (width 0.508) (layer F.Cu) (net 1))
-  (segment (start 169.037 89.281) (end 169.037 94.361) (width 0.508) (layer F.Cu) (net 1))
-  (segment (start 168.148 88.392) (end 169.037 89.281) (width 0.508) (layer F.Cu) (net 1))
-  (segment (start 167.386 88.392) (end 168.148 88.392) (width 0.508) (layer F.Cu) (net 1))
-  (segment (start 166.636 87.642) (end 167.386 88.392) (width 0.508) (layer F.Cu) (net 1))
   (segment (start 162.941 110.986) (end 162.941 115.062) (width 0.508) (layer F.Cu) (net 1))
   (segment (start 161.036 116.967) (end 155.448 116.967) (width 0.508) (layer F.Cu) (net 1))
