File: KiCAD/RGBLLSC.sch (KiCad schematic (older format))
At the start: 16 parts, among them P1 PICKIT3, P2 RGB-LED-Strip, Q1 FQP30N06L, Q2 FQP30N06L, Q3 FQP30N06L, U1 PIC12F1840

Commit message: Updated Schematic
Parts:
- removed P2: RGB-LED-Strip, symbol CONN_01X04
- removed P?: I2C, symbol CONN_01X02
- added D1: LED, symbol LED
- added P2: PWR IN, symbol CONN_01X03
- added P3: MAIN OUT, symbol CONN_01X06
- added R10, R9: 4.7K, symbol R
- added R7: R, symbol R
- gave numbers to parts that had none: 2
Connections:
- net +12V: now also P2.2 (P2), P3.3 (P3)
- net +5V: now also D1.2 (A); no longer C1.2, P1.2 (P2), R8.1, U1.1 (Vdd)
- net GND: now also P2.3 (P3), R7.2
- net at Q2.2 (D): now also P3.5 (P5)
- net at U1.5 (RA2/AN2/SDA): now also P3.2 (P2), R10.2
- net at P1.5 (P5), U1.6 (RA1/AN1/PGC/SCL): now also P3.1 (P1), R9.2
- net at Q1.2 (D): now also P3.4 (P4)
- net at Q3.2 (D): now also P3.6 (P6)
- new net: D1.1 (K), R7.1
- new net +3V3: C1.2, P1.2 (P2), P2.1 (P1), R10.1, R8.1, R9.1, U1.1 (Vdd)
Other:
- note added: "Main Circuit Board"
- note added: "NOTES:"
- note added: "Screw Terminal\n"
- note added: "WARNING: Do NOT program \nthe device while anything is \npluged into it"
- moved on the sheet: C1, P1, Q1, Q2, Q3, R1, R2, R3, R4, R5, R6, R8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

Commit message: Updated PCB Design and Schematic
Parts:
- C1: footprint (none) -> Capacitors_SMD:C_0603
- D1: footprint (none) -> LEDs:LED_0603
- P1: footprint (none) -> Pin_Headers:Pin_Header_Straight_1x06
- P3: footprint (none) -> User:Screw-Terminal-Thingy-5.08mm-0.2in
- Q1, Q2, Q3: footprint (none) -> TO_SOT_Packages_THT:TO-220_Neutral123_Vertical
- R1, R10, R2, R3, R4, R5, R6, R7, R8, R9: footprint (none) -> Resistors_SMD:R_0603
- SW1: footprint (none) -> Buttons_Switches_ThroughHole:SW_TH_Tactile_Omron_B3F-10xx
- U1: footprint (none) -> Housings_DIP:DIP-8_W7.62mm_LongPads
Connections:
- net +12V: now also P3.4 (P4); no longer P3.3 (P3)
- net at Q2.2 (D): now also P3.2 (P2); no longer P3.5 (P5)
- net at P1.5 (P5), U1.6 (RA1/AN1/PGC/SCL): now also P3.5 (P5), R10.2; no longer P3.1 (P1), R9.2
- net at Q1.2 (D): now also P3.3 (P3); no longer P3.4 (P4)
- net at P3.6 (P6): now also R9.2, U1.5 (RA2/AN2/SDA); no longer Q3.2 (D)
- new net: P3.1 (P1), Q3.2 (D)

Commit message: Finished PCB
Parts:
- P2: footprint (none) -> User:Screw-Terminal-Thingy-3pin-3.5mm
- P3: footprint User:Screw-Terminal-Thingy-5.08mm-0.2in -> User:Screw-Terminal-Thingy-6pin-3.5mm
Connections:
- net +3V3 is gone; now on net +5V: C1.2, P1.2 (P2), P2.1 (P1), R10.1, R8.1, R9.1, U1.1 (Vdd)
Changed lines of the file:
@@
-	1    0    0    -1
-$EndComp
-$Comp
-L +3.3V #PWR08
-U 1 1 56A8C0EE
-P 4900 1550
-F 0 "#PWR08" H 4900 1400 50  0001 C CNN
-F 1 "+3.3V" H 4900 1690 50  0000 C CNN
-F 2 "" H 4900 1550 50  0000 C CNN
-F 3 "" H 4900 1550 50  0000 C CNN
-	1    4900 1550
-	1    0    0    -1
-$EndComp
-$Comp
-L +3.3V #PWR09
-U 1 1 56A8C4D0
-P 4100 1400
-F 0 "#PWR09" H 4100 1250 50  0001 C CNN
-F 1 "+3.3V" H 4100 1540 50  0000 C CNN
-F 2 "" H 4100 1400 50  0000 C CNN
-F 3 "" H 4100 1400 50  0000 C CNN
-	1    4100 1400
-	1    0    0    -1
-$EndComp
-$Comp
-L +3.3V #PWR010
-U 1 1 56A8C511
-P 1500 1400
-F 0 "#PWR010" H 1500 1250 50  0001 C CNN
-F 1 "+3.3V" H 1500 1540 50  0000 C CNN
-F 2 "" H 1500 1400 50  0000 C CNN
-F 3 "" H 1500 1400 50  0000 C CNN
-	1    1500 1400
-	1    0    0    -1
-$EndComp
-$Comp
-L +3.3V #PWR011
-U 1 1 56A8C565
-P 2300 1450
-F 0 "#PWR011" H 2300 1300 50  0001 C CNN
-F 1 "+3.3V" H 2300 1590 50  0000 C CNN
-F 2 "" H 2300 1450 50  0000 C CNN
-F 3 "" H 2300 1450 50  0000 C CNN
-	1    2300 1450
 	1    0    0    -1
 $EndComp
@@
 WARNING: Do NOT program \nthe device while anything is \npluged into it
 $Comp
-L GND #PWR012
+L GND #PWR08
 U 1 1 56A8D38D
 P 1300 3050
-F 0 "#PWR012" H 1300 2800 50  0001 C CNN
+F 0 "#PWR08" H 1300 2800 50  0001 C CNN
 F 1 "GND" H 1300 2900 50  0000 C CNN
 F 2 "" H 1300 3050 50  0000 C CNN
@@
 	1    0    0    -1
 $EndComp
-$Comp
-L +3.3V #PWR013
-U 1 1 56A8D528
-P 1300 2850
-F 0 "#PWR013" H 1300 2700 50  0001 C CNN
-F 1 "+3.3V" H 1300 2990 50  0000 C CNN
-F 2 "" H 1300 2850 50  0000 C CNN
-F 3 "" H 1300 2850 50  0000 C CNN
-	1    1300 2850
-	1    0    0    -1
-$EndComp
-Wire Wire Line
-	3800 1700 4250 1700
-Wire Wire Line
-	4250 1700 4350 1700
-Wire Wire Line
-	3800 1600 4100 1600
-Wire Wire Line
-	4100 1600 4350 1600
-Wire Wire Line
-	3800 1500 3900 1500
-Wire Wire Line
-	3900 1500 4350 1500
+Wire Wire Line
+	3800 1700 4350 1700
+Wire Wire Line
+	3800 1600 4350 1600
+Wire Wire Line
+	3800 1500 4350 1500
 Wire Wire Line
 	4350 1400 4100 1400
@@
 	1700 1800 1700 1150
 Wire Wire Line
-	1450 1800 1500 1800
-Wire Wire Line
-	1500 1800 1700 1800
-Wire Wire Line
-	1700 1800 2300 1800
+	1450 1800 2300 1800
 Wire Wire Line
 	1850 1500 1900 1500
@@
 	3100 2700 3050 2700
 Wire Wire Line
-	3050 2200 3050 2700
-Wire Wire Line
-	3050 2700 3050 2750
+	3050 2200 3050 2750
 Wire Wire Line
 	3050 3050 3050 3100
 Wire Wire Line
-	3050 3100 3400 3100
-Wire Wire Line
-	3400 3100 3750 3100
+	3050 3100 3750 3100
 Wire Wire Line
 	3750 3100 3750 2900
@@
 	2050 2700 2000 2700
 Wire Wire Line
-	2000 2200 2000 2700
-Wire Wire Line
-	2000 2700 2000 2750
+	2000 2200 2000 2750
 Wire Wire Line
 	2000 3050 2000 3100
 Wire Wire Line
-	2000 3100 2350 3100
-Wire Wire Line
-	2350 3100 2700 3100
+	2000 3100 2700 3100
 Wire Wire Line
 	2700 3100 2700 2900
@@
 	4100 3050 4100 3100
 Wire Wire Line
-	4100 3100 4450 3100
-Wire Wire Line
-	4450 3100 4800 3100
+	4100 3100 4800 3100
 Wire Wire Line
 	4800 3100 4800 2900
@@
 	3800 1800 3800 1800
 Wire Wire Line
-	4100 1600 4100 2700
-Wire Wire Line
-	4100 2700 4100 2750
+	4100 1600 4100 2750
 Connection ~ 4100 1600
 Wire Wire Line
@@
 	4800 1650 4800 1600
 Wire Wire Line
-	4800 1600 4900 1600
-Wire Wire Line
-	4900 1600 5000 1600
+	4800 1600 5000 1600
 Wire Wire Line
 	5000 1600 5000 1650
@@
 	5700 1400 5700 1100
 $Comp
-L +12V #PWR014
+L +12V #PWR09
 U 1 1 56A8E224
 P 1450 2950
-F 0 "#PWR014" H 1450 2800 50  0001 C CNN
+F 0 "#PWR09" H 1450 2800 50  0001 C CNN
 F 1 "+12V" H 1450 3090 50  0000 C CNN
 F 2 "" H 1450 2950 50  0000 C CNN
@@
 F 0 "P2" H 1050 3150 50  0000 C CNN
 F 1 "PWR IN" V 1150 2950 50  0000 C CNN
-F 2 "" H 1050 2950 50  0001 C CNN
+F 2 "User:Screw-Terminal-Thingy-3pin-3.5mm" H 1050 2950 50  0001 C CNN
 F 3 "" H 1050 2950 50  0000 C CNN
 	1    1050 2950
@@
 F 0 "P3" H 5450 2600 50  0000 C CNN
 F 1 "MAIN OUT" V 5550 2250 50  0000 C CNN
-F 2 "User:Screw-Terminal-Thingy-5.08mm-0.2in" H 5450 2250 50  0001 C CNN
+F 2 "User:Screw-Terminal-Thingy-6pin-3.5mm" H 5450 2250 50  0001 C CNN
 F 3 "" H 5450 2250 50  0000 C CNN
 	1    5450 2250
@@
 $EndComp
 $Comp
-L GND #PWR015
+L GND #PWR010
 U 1 1 56A98131
 P 900 2200
-F 0 "#PWR015" H 900 1950 50  0001 C CNN
+F 0 "#PWR010" H 900 1950 50  0001 C CNN
 F 1 "GND" H 900 2050 50  0000 C CNN
 F 2 "" H 900 2200 50  0000 C CNN
@@
 $EndComp
 $Comp
-L +5V #PWR016
+L +5V #PWR011
 U 1 1 56A9816D
 P 1750 2200
-F 0 "#PWR016" H 1750 2050 50  0001 C CNN
+F 0 "#PWR011" H 1750 2050 50  0001 C CNN
 F 1 "+5V" H 1750 2340 50  0000 C CNN
 F 2 "" H 1750 2200 50  0000 C CNN
@@
 	950  2200 900  2200
 Wire Wire Line
-	5250 2100 5000 2100
-Wire Wire Line
-	5000 2100 4250 2100
+	4250 2100 5250 2100
 Wire Wire Line
 	4250 2100 4250 1700
 Connection ~ 4250 1700
 Wire Wire Line
-	5250 2000 4800 2000
-Wire Wire Line
-	4800 2000 3800 2000
+	3800 2000 5250 2000
 Wire Wire Line
 	3800 2000 3800 1800
+$Comp
+L +5V #PWR012
+U 1 1 56AA6AC4
+P 2300 1450
+F 0 "#PWR012" H 2300 1300 50  0001 C CNN
+F 1 "+5V" H 2300 1590 50  0000 C CNN
+F 2 "" H 2300 1450 50  0000 C CNN
+F 3 "" H 2300 1450 50  0000 C CNN
+	1    2300 1450
+	1    0    0    -1
+$EndComp
+$Comp
+L +5V #PWR013
+U 1 1 56AA6B0B
+P 1500 1400
+F 0 "#PWR013" H 1500 1250 50  0001 C CNN
+F 1 "+5V" H 1500 1540 50  0000 C CNN
+F 2 "" H 1500 1400 50  0000 C CNN
+F 3 "" H 1500 1400 50  0000 C CNN
+	1    1500 1400
+	1    0    0    -1
+$EndComp
+$Comp
+L +5V #PWR014
+U 1 1 56AA6B52
+P 4100 1400
+F 0 "#PWR014" H 4100 1250 50  0001 C CNN
+F 1 "+5V" H 4100 1540 50  0000 C CNN
+F 2 "" H 4100 1400 50  0000 C CNN
+F 3 "" H 4100 1400 50  0000 C CNN
+	1    4100 1400
+	1    0    0    -1
+$EndComp
+$Comp
+L +5V #PWR015
+U 1 1 56AA6B99
+P 4900 1550
+F 0 "#PWR015" H 4900 1400 50  0001 C CNN
+F 1 "+5V" H 4900 1690 50  0000 C CNN
+F 2 "" H 4900 1550 50  0000 C CNN
+F 3 "" H 4900 1550 50  0000 C CNN
+	1    4900 1550
+	1    0    0    -1
+$EndComp
+$Comp
+L +5V #PWR016
+U 1 1 56AA6BE0
+P 1300 2850
+F 0 "#PWR016" H 1300 2700 50  0001 C CNN
+F 1 "+5V" H 1300 2990 50  0000 C CNN
+F 2 "" H 1300 2850 50  0000 C CNN
+F 3 "" H 1300 2850 50  0000 C CNN
+	1    1300 2850
+	1    0    0    -1
+$EndComp
 $EndSCHEMATC

Commit message: Added Project Images
Parts:
- R7: value R -> 470
Other:
- note added: "Main Input\n"
- note removed: "Screw Terminal\n"
Changed lines of the file:
@@
 	1    0    0    -1
 $EndComp
-Text Notes 850  2600 0    60   ~ 0
-Screw Terminal\n
 Wire Notes Line
 	800  2450 800  3300
@@
 P 1100 2200
 F 0 "R7" V 1180 2200 50  0000 C CNN
-F 1 "R" V 1100 2200 50  0000 C CNN
+F 1 "470" V 1100 2200 50  0000 C CNN
 F 2 "Resistors_SMD:R_0603" V 1030 2200 50  0001 C CNN
 F 3 "" H 1100 2200 50  0000 C CNN
@@
 	1    0    0    -1
 $EndComp
+Text Notes 950  2550 0    60   ~ 0
+Main Input\n
 $EndSCHEMATC
